Commit message: Driver now actually publishes IMU data instead of just creating the publisher and discarding everything

File: go2_description/urdf/go2_description.urdf (robot description, URDF)
Before this commit: robot go2_description, 30 links, 29 joints
Links:
- removed link radar
- added link utlidar_lidar, mass 0
Joints:
- removed joint radar_joint
- added joint utlidar_joint: type fixed, parent base_link, child utlidar_lidar, origin xyz=0.28945 0 -0.046825 rpy=0 2.8782 0, axis 0 0 0
