Commit message: Fix hesai lidar frame name

File: go2_description/urdf/lidar_4D_lidar.xacro (robot description, xacro)
@@ -2,5 +2,5 @@
 <robot xmlns:xacro="http://www.ros.org/wiki/xacro">
     <!-- Lidar L1-->
-    <link name="lidar_l1_link">
+    <link name="hesai_lidar">
         <inertial>
             <mass value="0.5"/>
@@ -27,12 +27,12 @@
         </collision>
     </link>
-    <joint name="lidar_l1_joint" type="fixed">
+    <joint name="hesai_lidar_joint" type="fixed">
         <parent link="base_link"/>
-        <child link="lidar_l1_link"/>
+        <child link="hesai_lidar"/>
         <!-- <origin rpy="2.94 0 1.5705" xyz="0.25 -0.038 -0.03"/> -->
         <origin rpy="2.879 0.0 1.5705" xyz="0.25 -0.038 -0.03"/>
     </joint>
-    <gazebo reference="lidar_l1_link">
-        <sensor name="lidar_l1" type="gpu_lidar">
+    <gazebo reference="hesai_lidar">
+        <sensor name="hesai_lidar" type="gpu_lidar">
             <topic>unitree_lidar</topic>
             <update_rate>10</update_rate>
@@ -64,5 +64,5 @@
             </lidar>
             <visualize>false</visualize>
-            <gz_frame_id>lidar_l1_link</gz_frame_id>
+            <gz_frame_id>hesai_lidar</gz_frame_id>
             <always_on>1</always_on>
         </sensor>

File: go2_description/urdf/unitree_go2_robot.xacro (robot description, xacro)
@@ -114,10 +114,10 @@
         <origin rpy="0 0 0" xyz="0.326 0 0.043" />
     </joint>
-    <!-- <joint name="lidar_l1_joint" type="fixed">
+    <!-- <joint name="hesai_lidar_joint" type="fixed">
         <parent link="base_link"/>
-        <child link="lidar_l1_link"/>
+        <child link="hesai_lidar"/>
         <origin rpy="2.94 0 1.5705" xyz="0.25 -0.038 -0.03"/>
     </joint>
-    <link name="lidar_l1_link">
+    <link name="hesai_lidar">
         <inertial>
             <mass value="0.5"/>
