Commit message: Lidar tilt

File: go2_description/urdf/hesai_lidar.xacro (robot description, xacro)
@@ -1,10 +1,19 @@
 <?xml version="1.0"?>
 <robot xmlns:xacro="http://www.ros.org/wiki/xacro">
-    <joint name="velodyne_base_mount_joint" type="fixed">
-        <origin rpy="0 0 0" xyz="0.2 0 0.08"/>
-        <parent link="base_link"/>
-        <child link="velodyne_base_link"/>
-    </joint>
-    <link name="velodyne_base_link">
+    <xacro:if value="$(arg tilted_lidar)">
+        <joint name="hesai_base_mount_joint" type="fixed">
+            <origin rpy="0.0 0.78539815 0.0" xyz="0.2 0 0.22"/>
+            <parent link="base_link"/>
+            <child link="hesai_base_link"/>
+        </joint>
+    </xacro:if>
+    <xacro:unless value="$(arg tilted_lidar)">
+        <joint name="hesai_base_mount_joint" type="fixed">
+            <origin rpy="0 0 0" xyz="0.2 0 0.08"/>
+            <parent link="base_link"/>
+            <child link="hesai_base_link"/>
+        </joint>
+    </xacro:unless>
+    <link name="hesai_base_link">
         <inertial>
             <mass value="0.83"/>
@@ -29,10 +38,10 @@
         </collision>
     </link>
-    <joint name="velodyne_base_scan_joint" type="fixed">
+    <joint name="hesai_base_scan_joint" type="fixed">
         <origin rpy="0 0 0" xyz="0 0 0.0377"/>
-        <parent link="velodyne_base_link"/>
-        <child link="velodyne"/>
+        <parent link="hesai_base_link"/>
+        <child link="hesai_lidar"/>
     </joint>
-    <link name="velodyne">
+    <link name="hesai_lidar">
         <inertial>
             <mass value="0.01"/>
@@ -48,9 +57,9 @@
     </link>
     <!-- Gazebo Sim Velodyne Sensor plugin -->
-    <gazebo reference="velodyne">
-        <sensor name="velodyne-VLP16" type="gpu_lidar">
-            <topic>velodyne_points</topic>
+    <gazebo reference="hesai_lidar">
+        <sensor name="hesai_lidar" type="gpu_lidar">
+            <topic>hesai_lidar</topic>
             <update_rate>10</update_rate>
-            <gz_frame_id>velodyne</gz_frame_id>
+            <gz_frame_id>hesai_lidar</gz_frame_id>
             <lidar>
                 <scan>
@@ -78,5 +87,5 @@
                     <stddev>0.008</stddev>
                 </noise>
-                <frame_id>velodyne</frame_id>
+                <frame_id>hesai_lidar</frame_id>
             </lidar>
             <visualize>true</visualize>

File: go2_description/urdf/unitree_go2_robot.xacro (robot description, xacro)
@@ -5,4 +5,5 @@
     <xacro:arg name="robot_controllers" default="$(find go2_description)/config/ros_control/ros_control.yaml"/>
     <xacro:arg name="robot_ns" default=""/>
+    <xacro:arg name="tilted_lidar" default="false"/>
     <xacro:include filename="$(find go2_description)/urdf/const.xacro" />
     <xacro:include filename="$(find go2_description)/urdf/materials.xacro" />
@@ -11,6 +12,6 @@
     <xacro:include filename="$(find go2_description)/urdf/unitree_go2_gazebo.xacro" />
     <!-- <xacro:include filename="$(find go2_description)/launch/stairs.urdf.xacro"/> -->
-    <xacro:include filename="$(find go2_description)/urdf/velodyne.xacro"/>
-    <xacro:include filename="$(find go2_description)/urdf/lidar_4D_lidar.xacro"/>
+    <xacro:include filename="$(find go2_description)/urdf/hesai_lidar.xacro"/>
+    <xacro:include filename="$(find go2_description)/urdf/unitree_lidar.xacro"/>
     <xacro:include filename="$(find go2_description)/urdf/realsense_d455.xacro"/>
     <!-- <xacro:stairs stairs="15" xpos="0" ypos="0" zpos="0" /> -->
@@ -114,34 +115,4 @@
         <origin rpy="0 0 0" xyz="0.326 0 0.043" />
     </joint>
-    <!-- <joint name="hesai_lidar_joint" type="fixed">
-        <parent link="base_link"/>
-        <child link="hesai_lidar"/>
-        <origin rpy="2.94 0 1.5705" xyz="0.25 -0.038 -0.03"/>
-    </joint>
-    <link name="hesai_lidar">
-        <inertial>
-            <mass value="0.5"/>
-            <origin rpy="0 0 0" xyz="0 0 0"/>
-            <inertia ixx="0.01" ixy="0" ixz="0" iyy="0.01" iyz="0" izz="0.01"/>
-        </inertial>
-        <visual>
-            <origin rpy="0 0 0" xyz="0 0 0"/>
-            <geometry>
-                <mesh filename="file://$(find go2_description)/meshes/L1_4D_Lidar.dae" scale="1 1 1"/>
-            </geometry>
-            <material name="black">
-                <color rgba="0.0 0.0 0.0 1.0"/>
-            </material>
-        </visual>
-        <collision>
-            <origin rpy="0 0 0" xyz="0 0 0"/>
-            <geometry>
-                <mesh filename="file://$(find go2_description)/meshes/L1_4D_Lidar.dae" scale="1 1 1"/>
-            </geometry>
-            <material name="black">
-                <color rgba="0.0 0.0 0.0 1.0"/>
-            </material>
-        </collision>
-    </link> -->
     <xacro:leg name="FR" mirror="-1" mirror_dae="False" front_hind="1" front_hind_dae="True" />
     <xacro:leg name="FL" mirror="1" mirror_dae="True" front_hind="1" front_hind_dae="True" />

File: go2_description/urdf/unitree_lidar.xacro (robot description, xacro)
@@ -2,5 +2,5 @@
 <robot xmlns:xacro="http://www.ros.org/wiki/xacro">
     <!-- Lidar L1-->
-    <link name="hesai_lidar">
+    <link name="unitree_lidar">
         <inertial>
             <mass value="0.5"/>
@@ -27,12 +27,12 @@
         </collision>
     </link>
-    <joint name="hesai_lidar_joint" type="fixed">
+    <joint name="unitree_lidar_joint" type="fixed">
         <parent link="base_link"/>
-        <child link="hesai_lidar"/>
+        <child link="unitree_lidar"/>
         <!-- <origin rpy="2.94 0 1.5705" xyz="0.25 -0.038 -0.03"/> -->
         <origin rpy="2.879 0.0 1.5705" xyz="0.25 -0.038 -0.03"/>
     </joint>
-    <gazebo reference="hesai_lidar">
-        <sensor name="hesai_lidar" type="gpu_lidar">
+    <gazebo reference="unitree_lidar">
+        <sensor name="unitree_lidar" type="gpu_lidar">
             <topic>unitree_lidar</topic>
             <update_rate>10</update_rate>
@@ -64,5 +64,5 @@
             </lidar>
             <visualize>false</visualize>
-            <gz_frame_id>hesai_lidar</gz_frame_id>
+            <gz_frame_id>unitree_lidar</gz_frame_id>
             <always_on>1</always_on>
         </sensor>

Commit message: Move lidar

File: go2_description/urdf/hesai_lidar.xacro (robot description, xacro)
@@ -3,5 +3,5 @@
     <xacro:if value="$(arg tilted_lidar)">
         <joint name="hesai_base_mount_joint" type="fixed">
-            <origin rpy="0.0 0.78539815 0.0" xyz="0.2 0 0.22"/>
+            <origin rpy="0.0 0.6 0.0" xyz="0.3 0 0.1"/>
             <parent link="base_link"/>
             <child link="hesai_base_link"/>
@@ -73,6 +73,6 @@
                         <samples>16</samples>
                         <resolution>1</resolution>
-                        <min_angle>-0.261799</min_angle>
-                        <max_angle>0.261799</max_angle>
+                        <min_angle>-0.3490659</min_angle>
+                        <max_angle>0.3490659</max_angle>
                     </vertical>
                 </scan>

Commit message: adds camera conf and lidar changes

File: go2_description/urdf/hesai_lidar.xacro (robot description, xacro)
@@ -3,5 +3,5 @@
     <xacro:if value="$(arg tilted_lidar)">
         <joint name="hesai_base_mount_joint" type="fixed">
-            <origin rpy="0.0 0.6 0.0" xyz="0.3 0 0.1"/>
+            <origin rpy="0.78 0.0 1.57" xyz="0.20 0 0.12"/>
             <parent link="base_link"/>
             <child link="hesai_base_link"/>
